File: usb-c-cable/usb-c-cable.sch (KiCad schematic (older format))
At the start: 5 parts, among them P1 USB_C_Plug, P2 USB_C_Plug

Commit message: represent B6 B7 pins on plug
Parts:
- P1, P2: symbol USB_C_Plug -> USB_C_Plug-RESCUE-usb-c-cable
- U?: value mcu -> internal mcu
Changed lines of the file:
@@
 EESchema Schematic File Version 2
+LIBS:usb-c-cable-rescue
 LIBS:power
 LIBS:device
@@
 $EndDescr
 $Comp
-L USB_C_Plug P2
+L USB_C_Plug-RESCUE-usb-c-cable P2
 U 1 1 5A246E8F
 P 4900 2200
@@
 Connection ~ 1075 3800
 Wire Wire Line
-	1775 1900 4300 1900
+	1775 1800 4300 1800
 Wire Wire Line
 	1775 1700 4300 1700
@@
 P 3125 1650
 F 0 "U?" H 2825 1650 60  0001 C CNN
-F 1 "mcu" H 3125 1725 60  0000 C CNN
+F 1 "internal mcu" H 3125 1725 60  0000 C CNN
 F 2 "" H 3125 1650 60  0001 C CNN
 F 3 "" H 3125 1650 60  0001 C CNN
@@
 	5200 3900 5200 3800
 $Comp
-L USB_C_Plug P1
+L USB_C_Plug-RESCUE-usb-c-cable P1
 U 1 1 5A246EFB
 P 1175 2200
@@
 	4300 3400 3150 3400
 Wire Wire Line
-	1775 3500 2900 3500
-Wire Wire Line
-	1775 3400 2900 3400
-Wire Wire Line
-	2900 3400 3150 3500
-Wire Wire Line
-	2900 3500 3150 3400
-Wire Wire Line
-	3175 3100 4300 3100
-Wire Wire Line
-	4300 3200 3150 3200
-Wire Wire Line
-	3175 3100 2900 2800
+	1775 3500 2925 3500
+Wire Wire Line
+	1775 3400 2925 3400
+Wire Wire Line
+	2925 3400 3150 3500
+Wire Wire Line
+	2925 3500 3150 3400
+Wire Wire Line
+	3200 3100 4300 3100
+Wire Wire Line
+	4300 3200 3175 3200
+Wire Wire Line
+	3200 3100 2900 2800
 Wire Wire Line
 	2900 2800 1775 2800
@@
 	1775 2900 2875 2900
 Wire Wire Line
-	2875 2900 3150 3200
-Wire Wire Line
-	1775 3100 2900 3100
-Wire Wire Line
-	2900 3100 3125 2800
-Wire Wire Line
-	3125 2800 4300 2800
-Wire Wire Line
-	1775 3200 2925 3200
-Wire Wire Line
-	2925 3200 3175 2900
-Wire Wire Line
-	3175 2900 4300 2900
-Wire Wire Line
-	3175 2500 4300 2500
-Wire Wire Line
-	4300 2600 3150 2600
-Wire Wire Line
-	3175 2500 2900 2200
+	2875 2900 3175 3200
+Wire Wire Line
+	1775 3100 2875 3100
+Wire Wire Line
+	2875 3100 3175 2800
+Wire Wire Line
+	3175 2800 4300 2800
+Wire Wire Line
+	1775 3200 2900 3200
+Wire Wire Line
+	2900 3200 3200 2900
+Wire Wire Line
+	3200 2900 4300 2900
+Wire Wire Line
+	3200 2500 4300 2500
+Wire Wire Line
+	4300 2600 3175 2600
+Wire Wire Line
+	3200 2500 2900 2200
 Wire Wire Line
 	2900 2200 1775 2200
@@
 	1775 2300 2875 2300
 Wire Wire Line
-	2875 2300 3150 2600
-Wire Wire Line
-	1775 2500 2900 2500
-Wire Wire Line
-	2900 2500 3125 2200
-Wire Wire Line
-	3125 2200 4300 2200
-Wire Wire Line
-	1775 2600 2925 2600
-Wire Wire Line
-	2925 2600 3175 2300
-Wire Wire Line
-	3175 2300 4300 2300
+	2875 2300 3175 2600
+Wire Wire Line
+	1775 2500 2875 2500
+Wire Wire Line
+	2875 2500 3175 2200
+Wire Wire Line
+	3175 2200 4300 2200
+Wire Wire Line
+	1775 2600 2900 2600
+Wire Wire Line
+	2900 2600 3200 2300
+Wire Wire Line
+	3200 2300 4300 2300
 $EndSCHEMATC
